Commit message: refactor the controller urdf to meet ros2_control mech; use scaled controller

File: src/jaka_zu5_moveit_config/config/jaka_zu5.ros2_control.xacro (robot description, xacro)
@@ -1,61 +1,68 @@
 <?xml version="1.0"?>
 <robot xmlns:xacro="http://www.ros.org/wiki/xacro">
-    <xacro:macro name="jaka_zu5_ros2_control" params="name initial_positions_file use_gazebo use_rviz_sim">
-        <xacro:property name="initial_positions" value="${xacro.load_yaml(initial_positions_file)['initial_positions']}"/>
-        <ros2_control name="${name}" type="system">
-            <!-- Include hardware plugin conditionally if rviz in simulation mode is enabled -->
-            <hardware>
-              <xacro:if value="${use_gazebo}">
-                  <!-- <plugin>gazebo_ros2_control/GazeboSystem</plugin> -->
-                  <plugin>ign_ros2_control/IgnitionSystem</plugin>
-              </xacro:if>
-              <xacro:if value="${use_rviz_sim}">
-                  <plugin>mock_components/GenericSystem</plugin>
-              </xacro:if>
-            </hardware>
-            <!-- Joint interfaces generated for each joint -->
-            <joint name="joint_1">
-                <command_interface name="position"/>
-                <state_interface name="position">
-                  <param name="initial_value">${initial_positions['joint_1']}</param>
-                </state_interface>
-                <state_interface name="velocity"/>
-            </joint>
-            <joint name="joint_2">
-                <command_interface name="position"/>
-                <state_interface name="position">
-                  <param name="initial_value">${initial_positions['joint_2']}</param>
-                </state_interface>
-                <state_interface name="velocity"/>
-            </joint>
-            <joint name="joint_3">
-                <command_interface name="position"/>
-                <state_interface name="position">
-                  <param name="initial_value">${initial_positions['joint_3']}</param>
-                </state_interface>
-                <state_interface name="velocity"/>
-            </joint>
-            <joint name="joint_4">
-                <command_interface name="position"/>
-                <state_interface name="position">
-                  <param name="initial_value">${initial_positions['joint_4']}</param>
-                </state_interface>
-                <state_interface name="velocity"/>
-            </joint>
-            <joint name="joint_5">
-                <command_interface name="position"/>
-                <state_interface name="position">
-                  <param name="initial_value">${initial_positions['joint_5']}</param>
-                </state_interface>
-                <state_interface name="velocity"/>
-            </joint>
-            <joint name="joint_6">
-                <command_interface name="position"/>
-                <state_interface name="position">
-                  <param name="initial_value">${initial_positions['joint_6']}</param>
-                </state_interface>
-                <state_interface name="velocity"/>
-            </joint>
-        </ros2_control>
-    </xacro:macro>
+	<xacro:macro name="jaka_zu5_ros2_control" params="name initial_positions_file use_gazebo use_rviz_sim">
+		<xacro:property name="initial_positions" value="${xacro.load_yaml(initial_positions_file)['initial_positions']}"/>
+		<ros2_control name="${name}" type="system">
+			<!-- Include hardware plugin conditionally if rviz in simulation mode is enabled -->
+			<hardware>
+				<xacro:if value="${use_gazebo}">
+					<!-- <plugin>gazebo_ros2_control/GazeboSystem</plugin> -->
+					<plugin>ign_ros2_control/IgnitionSystem</plugin>
+				</xacro:if>
+				<xacro:if value="${use_rviz_sim}">
+					<plugin>mock_components/GenericSystem</plugin>
+				</xacro:if>
+				<xacro:unless value="${use_gazebo or use_rviz_sim}">
+					<plugin>whi_arm_interface/WhiArmInterface</plugin>
+					<param name="hw_start_duration_seconds">0.2</param>
+					<param name="hw_stop_duration_seconds">1.0</param>
+					<param name="arm_series">jaka</param>
+					<param name="hw_config">/media/nvidia/nvme0n1pnvme0n1p1/ros2_ws/src/whi_arm_interface/config/hardware_jaka.yaml</param>
+				</xacro:unless>
+			</hardware>
+			<!-- Joint interfaces generated for each joint -->
+			<joint name="joint_1">
+				<command_interface name="position"/>
+				<state_interface name="position">
+					<param name="initial_value">${initial_positions['joint_1']}</param>
+				</state_interface>
+				<state_interface name="velocity"/>
+			</joint>
+			<joint name="joint_2">
+				<command_interface name="position"/>
+				<state_interface name="position">
+					<param name="initial_value">${initial_positions['joint_2']}</param>
+				</state_interface>
+				<state_interface name="velocity"/>
+			</joint>
+			<joint name="joint_3">
+				<command_interface name="position"/>
+				<state_interface name="position">
+					<param name="initial_value">${initial_positions['joint_3']}</param>
+				</state_interface>
+				<state_interface name="velocity"/>
+			</joint>
+			<joint name="joint_4">
+				<command_interface name="position"/>
+				<state_interface name="position">
+					<param name="initial_value">${initial_positions['joint_4']}</param>
+				</state_interface>
+				<state_interface name="velocity"/>
+			</joint>
+			<joint name="joint_5">
+				<command_interface name="position"/>
+				<state_interface name="position">
+					<param name="initial_value">${initial_positions['joint_5']}</param>
+				</state_interface>
+				<state_interface name="velocity"/>
+			</joint>
+			<joint name="joint_6">
+				<command_interface name="position"/>
+				<state_interface name="position">
+					<param name="initial_value">${initial_positions['joint_6']}</param>
+				</state_interface>
+				<state_interface name="velocity"/>
+			</joint>
+		</ros2_control>
+	</xacro:macro>
 </robot>
